File: batt.kicad_sch (KiCad schematic)
At the start: 26 parts

Commit message: Add files via upload
Parts:
- added C? (x2): 4.7 uF, symbol Device:C_Small
- added C?: 100 nF, symbol Device:C_Small
- added C?: 10 uF, symbol Device:C_Small
- added D?: LED, symbol Device:LED
- added J?: Screw_Terminal_01x02, symbol Connector:Screw_Terminal_01x02
- added R?: 0.01 Ω, symbol Device:R_Small
- added R? (x4): 10K, symbol Device:R_Small
- added R? (x2): 10, symbol Device:R_Small
- added R?: 4K7, symbol Device:R_Small
- added R?: 200K, symbol Device:R_Small
- added SW?: SLIDE_BATT_REMOVE, symbol Switch:SW_DIP_x01
- added TP?: TestPoint, symbol Connector:TestPoint
- D?: value D_Schottky_Small_Filled -> PMEG4050EP
- R?: value 910K -> 1M
Connections:
- net VBAT is gone; now on net +BATT: C?.2, D?.2 (A), J?.1, R?.1, U?.12 (BATT)
- net VSYS is gone; now on net VS: D?.1 (K), Q?.2 (S), U?.6 (SYS)
- net GND: now also C?.1, C?.2, C?.2, C?.1, C?.2, C?.2, R?.1, R?.2; no longer U?.13 (THM)
- net PVL: now also R?.1, R?.1
- net BATN: now reaches C?.2, J?.4, Q?.2 (S), R?.2
- net BATN: now also U?.10 (BATSN), J?.1 (Pin_1)
- net AVL: now reaches C?.2, R?.2, U?.26 (AVL)
- net AVL: now also SW?.2
- net VS: now reaches C?.1
- net VS: now also C?.1, C?.2, U?.19 (SYSA), C?.2
- net +BATT: now reaches U?.11 (BATSP)
- net +BATT: now also J?.2 (Pin_2)
- net STAT: now reaches U?.16 (STAT)
- net STAT: now also D?.1 (K)
- net INOKB: now reaches U?.17 (INOKB)
- net INOKB: now also R?.2, TP?.1
- net at U?.18 (INTB): now also R?.2
- net at U?.28 (STBY): now also R?.1
- net CSINP: now reaches U?.29 (CSINP)
- net CSINP: now also C?.1, C?.1, R?.1
- net CSINN: now reaches U?.30 (CSINN)
- net CSINN: now also C?.1, C?.2, R?.1
- net VPD renamed CHGIN
- net CHGIN: now also R?.2, R?.2
- new net: D?.2 (A), R?.2
- new net: R?.1, SW?.1
- new net +3V3: R?.1
- new net THM: R?.2, R?.2, U?.13 (THM)
- new net VD: R?.1, R?.2
- no-connect marks 1 -> 0
Other:
- note added: "3S Lipo Plug, JST Will probably not be placed Unfortunately, most JSTs lipo conns are cabled for low Amps"
- note added: "Datasheet had nothing on what CSINP and CSINN resistor values should be, used EVAL board as ref EVAL has 15nF caps on CSINP and CSINN"
- note added: "EVAL has 220K and 470K here datasheet has 470K and 910K"
- note added: "Hot Insertion Protection RC, copied from datasheet"
- note added: "LIPO Charging LED STAT goes high when no charge or no power Cycles low/high when charging and low when charged STAT tied to PVL with 200K in datasheet, no LED there I figured down to 10K LED should still be visible if very dim"
- note added: "Not using a thermistor. THM to GND means battery removal cannot be detected, but allows charging THM to AVL is equivalent to battery removal detection, and prevents charging"
- note added: "The slave address of the IC is 0xD2h/0xD3h The least significant bit is the read/write indicator (1 for read, 0 for write)"
- note added: "Using defaults for charge settings by tying to PVL don't need resistors for those"
- note added: "Vsys is guaranteed 4V - 14V Vsys should be between Vsysmin (8.4V programmable) to Vbattreg (12V, programmable)"
- note added: "Will use DMN3020, DMN3016, or similar, but this MOSFET works for draft"
- note removed: "3S Lipo Plug, JST"
- note removed: "Hot Insertion Protection RC"
- note removed: "Might need a higher Amp MOSFET"
- moved on the sheet: C?, L?, R?, U?

Commit message: production version (2023)
Parts:
- removed D?: LED, symbol Device:LED
- removed J?: Screw_Terminal_01x02, symbol Connector:Screw_Terminal_01x02
- removed J?: B4B-XH-AMLFSN, CONN_B4B-XH-AM_JST:B4B-XH-AMLFSN, symbol JST XH 4:B4B-XH-AMLFSN
- removed Q? (x3): AO3400A, Package_TO_SOT_SMD:SOT-23, symbol Transistor_FET:AO3400A
- removed R? (x2): 10K, symbol Device:R_Small
- removed R?: 470K, symbol Device:R_Small
- removed R?: 200K, symbol Device:R_Small
- removed SW?: SLIDE_BATT_REMOVE, symbol Switch:SW_DIP_x01
- added C35, C53: 10 nF 50V X7R, Capacitor_SMD:C_0402_1005Metric_Pad0.74x0.62mm_HandSolder, symbol Device:C_Small
- added C41: 10 uF 35V X7R, Capacitor_SMD:C_1206_3216Metric, symbol Device:C_Small
- added C51: 4.7 uF 16V X5R, Capacitor_SMD:C_0603_1608Metric_Pad1.08x0.95mm_HandSolder, symbol Device:C_Small
- added C52: 33 pF 6V C0G, Capacitor_SMD:C_0402_1005Metric_Pad0.74x0.62mm_HandSolder, symbol Device:C_Small
- added D10, D12: LED_GREEN, LED_SMD:LED_0603_1608Metric, symbol Device:LED
- added D11, D13, D18: PTVS22VS1UR, PowerIC:TVS_PTVS22VS1UR, symbol PTVS22VS1UR:PTVS22VS1UR
- added D15, D16: LED_BLUE, LED_SMD:LED_0603_1608Metric, symbol Device:LED
- added D17: D_Schottky, Diode_SMD:D_SMA, symbol Device:D_Schottky
- added F1: Fuse Holder, Fuse:Fuseholder_Blade_Mini_Keystone_3568, symbol Device:Fuse
- added J16: THM, Connector_PinHeader_2.54mm:PinHeader_1x02_P2.54mm_Vertical, symbol Connector:Conn_01x02_Female
- added J17: header, Connector_PinHeader_2.54mm:PinHeader_1x01_P2.54mm_Vertical, symbol Connector:Conn_01x01_Female
- added J20: XT60-M, PowerIC:AMASS_XT60-M, symbol XT60:XT60-M
- added JP4: AVL_JP, Jumper:SolderJumper-2_P1.3mm_Open_RoundedPad1.0x1.5mm, symbol Jumper:SolderJumper_2_Open
- added JP5: HEADER-3X04, PCA85:3X04, symbol AdaPCA9685:HEADER-3X04
- added JP6: Jumper_2_Open, Jumper:SolderJumper-2_P1.3mm_Open_RoundedPad1.0x1.5mm, symbol Jumper:Jumper_2_Open
- added Q4, Q6, Q7: DMP3007SCG, Package_SON:Diodes_PowerDI3333-8, symbol Transistor_FET:DMP3013SFV
- added Q5: BSS138, Package_TO_SOT_SMD:SOT-23, symbol Transistor_FET:AO3400A
- added R44, R60: 110K, Capacitor_SMD:C_0603_1608Metric, symbol Device:R_Small
- added R45, R52, R72: 10K, Capacitor_SMD:C_0402_1005Metric_Pad0.74x0.62mm_HandSolder, symbol Device:R_Small
- added R53: 0.01 Ω 3W, Resistor_SMD:R_2512_6332Metric, symbol Device:R_Small
- added R54, R55: 226K, Capacitor_SMD:C_0402_1005Metric_Pad0.74x0.62mm_HandSolder, symbol Device:R_Small
- added R56, R66: 17k8, Capacitor_SMD:C_0402_1005Metric_Pad0.74x0.62mm_HandSolder, symbol Device:R_Small
- added R58: 4K7, Resistor_SMD:R_0603_1608Metric_Pad0.98x0.95mm_HandSolder, symbol Device:R_Small
- added R63, R69: 1K, Capacitor_SMD:C_0402_1005Metric_Pad0.74x0.62mm_HandSolder, symbol Device:R_Small
- added R65, R67: 200K, Capacitor_SMD:C_0402_1005Metric_Pad0.74x0.62mm_HandSolder, symbol Device:R_Small
- added R70, R71: 10, Capacitor_SMD:C_0402_1005Metric_Pad0.74x0.62mm_HandSolder, symbol Device:R_Small
- added SW4: CK PCM12SMTR, Button_Switch_SMD:SW_SPDT_PCM12, symbol Switch:SW_SPDT
- added TP4: TestPoint, TestPoint:TestPoint_Pad_D1.5mm, symbol Connector:TestPoint
- added TP6: TestPoint, TestPoint:TestPoint_Pad_1.5x1.5mm, symbol Connector:TestPoint
- added TP7: TestPoint, TestPoint:TestPoint_Pad_2.0x2.0mm, symbol Connector:TestPoint
- C36, C37, C38: renamed from C?; value 47 uF -> 47 uF 25V X7R; footprint (none) -> Capacitor_SMD:C_1210_3225Metric; JCLPCB (none) -> C403725; Vendor (none) -> C403725
- C39: renamed from C?; value 100 nF -> 100 nF 25V X7R; footprint (none) -> Capacitor_SMD:C_0402_1005Metric; JCLPCB (none) -> C307331; Vendor (none) -> C307331
- C40, C46, C49: renamed from C?; value 10 uF -> 10 uF 35V X7R; footprint (none) -> Capacitor_SMD:C_1206_3216Metric; JCLPCB (none) -> C13585; Vendor (none) -> C13585
- C42, C43: renamed from C?; value 220 nF -> 220 nF 16V X7R; footprint (none) -> Capacitor_SMD:C_0402_1005Metric; JCLPCB (none) -> C16772; Vendor (none) -> C16772
- C44, C45: renamed from C?; value 4.7 uF -> 10 nF 50V X7R; footprint (none) -> Capacitor_SMD:C_0402_1005Metric_Pad0.74x0.62mm_HandSolder; JCLPCB (none) -> C15195; Vendor (none) -> C15195
- C47, C48: renamed from C?; value 4.7 uF -> 4.7 uF 16V X5R; footprint (none) -> Capacitor_SMD:C_0603_1608Metric_Pad1.08x0.95mm_HandSolder; JCLPCB (none) -> C19666; Vendor (none) -> C19666
- C50: renamed from C?; value 47 nF -> 47 nF 30V X7R; footprint (none) -> Capacitor_SMD:C_0603_1608Metric_Pad1.08x0.95mm_HandSolder; JCLPCB (none) -> C1622; Vendor (none) -> C1622
- D14: renamed from D?; value PMEG4050EP -> DNP; footprint (none) -> Diode_SMD:D_SOD-128
- J18, J19: renamed from J?; value Screw_Terminal_01x02 -> Terminal; footprint (none) -> TerminalBlock_Phoenix:TerminalBlock_Phoenix_MKDS-1,5-2-5.08_1x02_P5.08mm_Horizontal; JCLPCB (none) -> C8478; Vendor (none) -> C8478
- L1: renamed from L?; value 3.3 uH -> 3.3 uH DR127-3R3-R; footprint (none) -> Inductor_SMD:InductorSMMS1360; JCLPCB (none) -> C149526; Vendor (none) -> C149526
- R46: renamed from R?; value 4K7 -> 1K; footprint (none) -> Capacitor_SMD:C_0402_1005Metric_Pad0.74x0.62mm_HandSolder; JCLPCB (none) -> C11702; Vendor (none) -> C11702
- R47, R51: renamed from R?; footprint (none) -> Capacitor_SMD:C_0402_1005Metric_Pad0.74x0.62mm_HandSolder; JCLPCB (none) -> C25077; Vendor (none) -> C25077
- R48: renamed from R?; value 0.01 Ω -> 0.01 Ω 3W; footprint (none) -> Resistor_SMD:R_2512_6332Metric; JCLPCB (none) -> C500740; Vendor (none) -> C500740
- R49, R50, R57, R59: renamed from R?; footprint (none) -> Capacitor_SMD:C_0402_1005Metric_Pad0.74x0.62mm_HandSolder; JCLPCB (none) -> C25744; Vendor (none) -> C25744
- R61: renamed from R?; footprint (none) -> Capacitor_SMD:C_0603_1608Metric; JCLPCB (none) -> C23164; Vendor (none) -> C23164
- R62: renamed from R?; footprint (none) -> Capacitor_SMD:C_0402_1005Metric_Pad0.74x0.62mm_HandSolder; JCLPCB (none) -> C2684545; Vendor (none) -> C2684545
- R64: renamed from R?; footprint (none) -> Capacitor_SMD:C_0402_1005Metric_Pad0.74x0.62mm_HandSolder; JCLPCB (none) -> C11702; Vendor (none) -> C11702
- R68: renamed from R?; footprint (none) -> Capacitor_SMD:C_0402_1005Metric_Pad0.74x0.62mm_HandSolder; JCLPCB (none) -> C26083; Vendor (none) -> C26083
- TP5: renamed from TP?; footprint (none) -> TestPoint:TestPoint_Pad_D1.5mm
- U10: renamed from U?; value MAX77961EFV06+ -> MAX77960x06; JCLPCB (none) -> C1020018; Vendor (none) -> C1020018
Connections:
- net +5V: now also C51.1, Q4.1 (S), Q4.2 (S), Q4.3 (S), R66.1
- net +BATT: now also C53.1, F1.2, J20.P (POS), R67.1
- net AVL: now also JP4.1 (A), SW4.3 (C)
- net CHGIN: now also C41.2
- net GND: now also J19.2 (Pin_2), U10.10 (BATSN), C35.2, C41.1, C51.2, C52.1, C53.2, D11.A, D13.A, D15.1 (K), D16.1 (K), D17.2 (A), D18.A, J16.1 (Pin_1), JP5.12, JP5.3, JP5.6, JP5.9, Q5.2 (S), R44.2, R54.1, R55.1, R56.1, R60.1, TP6.1; no longer J19.1 (Pin_1)
- net INOKB: now also R58.1
- net LX1: now also L1.1, U10.3 (LX1)
- net MSFT_5V: now also Q5.1 (G)
- net PVL: now also JP6.2 (B); no longer U10.21 (INLIM), U10.23 (ISET), U10.24 (VSET), U10.25 (ITO)
- net STAT: now also R45.2, TP4.1
- net THM: now also J16.2 (Pin_2), R44.1, R52.1
- net VS: now also D11.C, J17.1 (Pin_1), JP5.11, JP5.2, JP5.5, JP5.8, R53.2; no longer C36.2, C37.1, C38.1, C46.2, D14.1 (K), U10.19 (SYSA), U10.6 (SYS)
- net 5V_MS: now reaches J18.2 (Pin_2)
- net 5V_MS: now also D13.C, Q4.5 (D), R63.1
- net BAT_SFS: now reaches C50.1, R64.1, R68.1
- net BAT_SFS: now also R65.2
- net CNFG: now reaches R62.2, U10.22 (CNFG)
- net CNFG: now also JP6.1 (A)
- net BST1: now reaches C43.2, U10.1 (BST1)
- net BST2: now reaches C42.1, U10.9 (BST2)
- net BT_G: now reaches R64.2
- net at R46.1: now also SW4.2 (B)
- net BATN renamed BT_S
- net BT_S: now also J20.N (NEG); no longer U10.10 (BATSN)
- new net: D12.1 (K), R58.2
- new net: Q7.4 (G), R71.2
- new net: R54.2, U10.24 (VSET)
- new net: R60.2, U10.23 (ISET)
- new net: D16.2 (A), R69.1
- new net: D15.2 (A), R63.2
- new net: R65.1, R67.2
- new net: R55.2, U10.25 (ITO)
- new net: Q6.4 (G), R70.2
- new net: D10.1 (K), R45.1
- new net +5VD: D10.2 (A), D12.2 (A)
- new net 5V_IMS: Q4.4 (G), Q5.3 (D), R66.2
- new net BATT_OUT: D17.1 (K), D18.C, J19.1 (Pin_1), Q6.5 (D), Q7.5 (D), R69.2, TP7.1
- new net FUSE_OUT: F1.1, Q6.1 (S), Q6.2 (S), Q6.3 (S), Q7.1 (S), Q7.2 (S), Q7.3 (S), R72.1
- new net HV_D: R70.1, R71.1, R72.2
- new net HV_G: C52.2
- new net INLIM: R56.2, U10.21 (INLIM)
- new net SYS_HEAD1: JP5.1
- new net SYS_HEAD2: JP5.4
- new net SYS_HEAD3: JP5.10, JP5.7
- new net THM_IN: JP4.2 (B), R52.2
- new net VPP: C35.1, C36.2, C37.1, C38.1, C46.2, D14.1 (K), R53.1, U10.19 (SYSA), U10.6 (SYS)
- no-connect marks 0 -> 1
Other:
- note added: "2S Lipo Selector"
- note added: "3S Lipo Plug, JST 3S ONLY"
- note added: "EVAL has 15nF caps on CSINP and CSINN, 10 nF used here"
- note added: "EVAL has 220K and 470K here datasheet has 470K and 910K I used 200K + 200K and 1M as used elsewhere already"
- note added: "Extra N-channel is needed to make it high 3.3V = on, GND = off"
- note added: "Extra header for XT60 connector (7.2 mm pitch) From other pin of terminal"
- note added: "FETS are Terminals, controlled by switch from MCU"
- note added: "Hot Insertion Protection RC, copied from datasheet DMN3016LFDE in EVAL, N-channel"
- note added: "LIPO Charging LED STAT goes high when no charge or no power Cycles low/high when charging and low when charged STAT tied to PVL with 200K in datasheet, no LED there"
- note added: "N-channel"
- note added: "No voltage is measured across the config resistors after powerup. The voltages are sampled at powerup and then each current source is disabled."
- note added: "P-channel"
- note added: "THM to GND means battery removal cannot be detected, but allows charging THM to AVL is equivalent to battery removal detection, and prevents charging This switch is here to assure safe removal of battery Optional thermistor, as shown can only detect too hot to charge unless THM to GND pull down is removed"
- note added: "TI has some nice alternatives but currently impossible to find bq25792"
- note added: "TVS good for surge suppression these TVS have some inductive load rev protection (500 mah) but the Schottky is needed for higher current reverse protection but Schottky has high leakage current"
- note added: "The primary distinction between an N-Channel and a P-Channel MOSFET is that the N-Channel is usually connected to the Ground (-) side of the load, while the P-Channel is connected to the VCC (+) side"
- note added: "Voltage/Power sensing resistor"
- note added: "Vsys is guaranteed 4V - 14V Vsys should be between Vsysmin (8.4V programmable) to Vbattreg (12V, programmable) Max Current 10A"
- note added: "lower the inductor DCR (DC resistance) is, the higher the buck-boost efficiency is DR127-3R3-R, SER2915, 7443320330"
- note removed: "3S Lipo Plug, JST Will probably not be placed Unfortunately, most JSTs lipo conns are cabled for low Amps"
- note removed: "Datasheet had nothing on what CSINP and CSINN resistor values should be, used EVAL board as ref EVAL has 15nF caps on CSINP and CSINN"
- note removed: "EVAL has 220K and 470K here datasheet has 470K and 910K"
- note removed: "Hot Insertion Protection RC, copied from datasheet"
- note removed: "LIPO Charging LED STAT goes high when no charge or no power Cycles low/high when charging and low when charged STAT tied to PVL with 200K in datasheet, no LED there I figured down to 10K LED should still be visible if very dim"
- note removed: "Not using a thermistor. THM to GND means battery removal cannot be detected, but allows charging THM to AVL is equivalent to battery removal detection, and prevents charging"
- note removed: "Using defaults for charge settings by tying to PVL don't need resistors for those"
- note removed: "Vsys is guaranteed 4V - 14V Vsys should be between Vsysmin (8.4V programmable) to Vbattreg (12V, programmable)"
- note removed: "Will use DMN3020, DMN3016, or similar, but this MOSFET works for draft"
- moved on the sheet: C40, C44, C45, C46, C47, C48, J18, J19, L1, R46, R57, R59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
