File: drivers.kicad_sch (KiCad schematic)
At the start: 32 parts

Commit message: production version (2023)
Parts:
- removed R?: 0, symbol Device:R_Small
- removed R?: 1K, symbol Device:R_Small
- removed R?: 4k7, symbol Device:R_Small
- removed R?: 10K, symbol Device:R_Small
- removed R?: 27R, symbol Device:R_Small
- added C57, C59, C65: 100 nF 25V X7R, Capacitor_SMD:C_0402_1005Metric, symbol Device:C_Small
- added C58: DNP, Capacitor_THT:CP_Radial_D10.0mm_P5.00mm, symbol Device:C_Polarized
- added C61, C62, C70, C74, C75: 10 nF 50V X7R, Capacitor_SMD:C_0402_1005Metric_Pad0.74x0.62mm_HandSolder, symbol Device:C_Small
- added C68, C76: 22 uF 25V X7R, Capacitor_SMD:C_1210_3225Metric_Pad1.33x2.70mm_HandSolder, symbol Device:C_Small
- added C78: 4.7 uF 16V X5R, Capacitor_SMD:C_0603_1608Metric_Pad1.08x0.95mm_HandSolder, symbol Device:C_Small
- added D19: PTVS22VS1UR, PowerIC:TVS_PTVS22VS1UR, symbol PTVS22VS1UR:PTVS22VS1UR
- added D20: LED_BLUE, LED_SMD:LED_0603_1608Metric, symbol Device:LED
- added J21: Terminal, TerminalBlock_Phoenix:TerminalBlock_Phoenix_MKDS-1,5-2-5.08_1x02_P5.08mm_Horizontal, symbol Connector:Screw_Terminal_01x02
- added J22: Conn_01x04_Female, Connector_PinHeader_2.54mm:PinHeader_1x04_P2.54mm_Vertical, symbol Connector:Conn_01x04_Female
- added JP7: HEADER-3X04, PCA85:3X04, symbol AdaPCA9685:HEADER-3X04
- added Q8: DMP3007SCG, Package_SON:Diodes_PowerDI3333-8, symbol Transistor_FET:DMP3013SFV
- added Q9: BSS138, Package_TO_SOT_SMD:SOT-23, symbol Transistor_FET:AO3400A
- added R73, R89: 17k8, Capacitor_SMD:C_0402_1005Metric_Pad0.74x0.62mm_HandSolder, symbol Device:R_Small
- added R74, R79, R81, R88: 10K, Capacitor_SMD:C_0402_1005Metric_Pad0.74x0.62mm_HandSolder, symbol Device:R_Small
- added R80: 1180, Resistor_SMD:R_0402_1005Metric_Pad0.72x0.64mm_HandSolder, symbol Device:R_Small
- added R87: 0R, Resistor_SMD:R_1206_3216Metric, symbol Device:R_Small
- added TP11: TestPoint, TestPoint:TestPoint_Pad_1.5x1.5mm, symbol Connector:TestPoint
- added TP12: TestPoint, TestPoint:TestPoint_Pad_2.0x2.0mm, symbol Connector:TestPoint
- added TP8, TP9: TestPoint, TestPoint:TestPoint_Pad_D1.0mm, symbol Connector:TestPoint
- added U11: INA219BxD, Package_SO:SOIC-8_3.9x4.9mm_P1.27mm, symbol Analog_ADC:INA219BxD
- added U13: TPD4EUSB30, Package_SON:USON-10_2.5x1.0mm_P0.5mm, symbol Power_Protection:TPD4EUSB30
- C54, C56: renamed from C?; value NP -> DNP; footprint (none) -> Capacitor_THT:CP_Radial_D10.0mm_P5.00mm
- C55: renamed from C?; value 220 pF -> DNP; footprint (none) -> Capacitor_SMD:C_0603_1608Metric
- C60: renamed from C?; value 100 nF -> 100 nF 25V X7R; footprint (none) -> Capacitor_SMD:C_0402_1005Metric; JCLPCB (none) -> C307331; Vendor (none) -> C307331
- C63, C64, C66, C67, C69, C71, C72, C77: renamed from C?; value 22 uF -> 22 uF 25V X7R; footprint (none) -> Capacitor_SMD:C_1210_3225Metric_Pad1.33x2.70mm_HandSolder; JCLPCB (none) -> C12891; Vendor (none) -> C12891
- C73: renamed from C?; value 1 uF -> 1 uF 50V X5R; footprint (none) -> Capacitor_SMD:C_0603_1608Metric; JCLPCB (none) -> C15849; Vendor (none) -> C15849
- J23, J25: renamed from J?; value Screw_Terminal_01x02 -> Terminal; footprint (none) -> TerminalBlock_Phoenix:TerminalBlock_Phoenix_MKDS-1,5-2-5.08_1x02_P5.08mm_Horizontal; JCLPCB (none) -> C8478; Vendor (none) -> C8478
- J24: renamed from J?; value Screw_Terminal_01x02 -> Terminal; footprint (none) -> Connector_PinHeader_2.54mm:PinHeader_1x02_P2.54mm_Vertical
- R75, R77, R83, R84, R85: renamed from R?; footprint (none) -> Capacitor_SMD:C_0402_1005Metric_Pad0.74x0.62mm_HandSolder; JCLPCB (none) -> C2684545; Vendor (none) -> C2684545
- R76, R78: renamed from R?; footprint (none) -> Resistor_SMD:R_0402_1005Metric_Pad0.72x0.64mm_HandSolder; JCLPCB (none) -> C346633; Vendor (none) -> C346633
- R82: renamed from R?; footprint (none) -> Resistor_SMD:R_0603_1608Metric_Pad0.98x0.95mm_HandSolder; JCLPCB (none) -> C23162; Vendor (none) -> C23162
- R86: renamed from R?; footprint (none) -> Capacitor_SMD:C_0402_1005Metric_Pad0.74x0.62mm_HandSolder; JCLPCB (none) -> C25764; Vendor (none) -> C25764
- TP10: renamed from TP?; footprint (none) -> TestPoint:TestPoint_Pad_D1.5mm
- U12: renamed from U?; value MPM54304GMN-0002 -> MPM54304-0002; JCLPCB (none) -> C9900037420; Vendor (none) -> C9900037420
Connections:
- net +1V8: now also C74.1, J22.4 (Pin_4)
- net +3V3: now also C65.2, C68.2, C75.1, C78.2, J22.2 (Pin_2), R79.1, U11.5 (VS), U13.2 (D1-); no longer R82.1
- net +5V: now also C57.1, C62.1, J22.1 (Pin_1), JP7.11, JP7.2, JP7.5, JP7.8, R87.2, U13.4 (D2+), U13.5 (D2-); no longer J23.2 (Pin_2)
- net +5VD: now also J23.2 (Pin_2), C59.1, C61.1, R87.1
- net EN: now also R73.2, R74.1
- net FB1: now also C57.2, TP8.1
- net FB2: now also C59.2, TP9.1
- net FB3: now also R82.1, R81.2; no longer R82.2
- net GND: now also R82.2, C58.2, C61.2, C62.2, C65.1, C68.1, C70.1, C74.2, C75.2, C76.1, C78.1, D19.A, D20.1 (K), J21.2 (Pin_2), J22.3 (Pin_3), JP7.12, JP7.3, JP7.6, JP7.9, Q9.2 (S), R74.2, TP11.1, U11.1 (A1), U11.2 (A0), U11.6 (GND), U13.3 (GND), U13.8 (GND)
- net I2C0_SCL: now also U11.4 (SCL)
- net I2C0_SDA: now also U11.3 (SDA)
- net VS: now also C58.1, C70.2, C76.2, Q8.1 (S), Q8.2 (S), Q8.3 (S), R73.1, R89.1
- net VCC: now reaches C73.1, R86.1, U12.25 (VCC)
- new net: R79.2, R80.1
- new net: R80.2, R81.1
- new net: D20.2 (A), R88.2
- new net 5V Logic: U13.1 (D1+)
- new net 5V_HEAD1: JP7.1
- new net 5V_HEAD2: JP7.4
- new net 5V_HEAD3: JP7.7
- new net 5V_HEAD4: JP7.10
- new net MSFT_VSV: Q9.1 (G)
- new net MS_VsV: D19.C, J21.1 (Pin_1), Q8.5 (D), R88.1, TP12.1
- new net VS out: U11.7 (IN-)
- new net VS+: U11.8 (IN+)
- new net VsV_IMS: Q8.4 (G), Q9.3 (D), R89.2
Other:
- note added: "CK PCM12SMTR"
- note added: "Filtering option: 27R to each Vm and 100 nF to 1 uF cap between Vm + and -"
- note added: "GPIO default is PG (power good) EVAL board shows PG to VCC with 100K I'm using 200K just for simpler BOM"
- note added: "This capacitor enables soft start, not required here"
- note added: "Useful: https://community.element14.com/products/roadtest/b/blog/posts/mps-mpm54304-evm-roadtest---snippets"
- note added: "Using same USB TVS to minimize unique parts"
- note added: "Voltage Dividers to set Buck V outs FB Voltage on must suffixes is 0.6 V which I assume is the same as Vref A feed-forward cap on these Vout to FB can be used Helpful when large current loads are present 33 nF is recommended"
- note added: "i2c address: 1000000 with gnd and gnd, 0x40"
- note removed: "FB Voltage on must suffixes is 0.6 V which I assume is the same as Vref A feed-forward cap on these Vout to FB can be used 33 nF is recommended"
- note removed: "GPIO default is PG (power good) EVAL board shows this to VCC with 100K I'm using 200K just for simpler BOM"
- note removed: "not sure about this capacitor, is necessary? size? I figure something small, reused from elsewhere, just to make sure the EN doesn't un-engage accidentally"
- moved on the sheet: C56, C71, C77, J23, J24, J25, R82
