File: mcu_sheet.kicad_sch (KiCad schematic)
At the start: 35 parts

Commit message: Add files via upload
Parts:
- added TP? (x3): TestPoint, symbol Connector:TestPoint
- R?: value 470R -> 1K
Connections:
- net SWCLK: now also TP?.1
- net SWDIO: now also TP?.1
- net at R?.1, SW?.A (P), SW?.A' (P1): now also TP?.1
Other:
- note added: "Pins 48 and 49 share a capacitor for easier layout per pico datasheet All inputs use 100 nF except VREG in/out"
- note added: "exact ordering may change for easier layout"
- note removed: "Pins 48 and 49 share a capacitor All inputs use 100 nF except VREG in/out"
Changed lines of the file:
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@@
   (junction (at 144.78 179.07) (diameter 0) (color 0 0 0 0)
+  )
+  (junction (at 132.08 177.8) (diameter 0) (color 0 0 0 0)
   )
   (junction (at 208.28 140.97) (diameter 0) (color 0 0 0 0)
@@
     (stroke (width 0) (type default) (color 0 0 0 0))
   )
-  (wire (pts (xy 74.93 167.64) (xy 86.36 167.64))
+  (wire (pts (xy 69.85 167.64) (xy 86.36 167.64))
     (stroke (width 0) (type default) (color 0 0 0 0))
   )
@@
     (effects (font (size 1.27 1.27)) (justify left bottom))
   )
-  (text "Pins 48 and 49 share a capacitor\nAll inputs use 100 nF except VREG in/out"
+  (text "Pins 48 and 49 share a capacitor\nfor easier layout per pico datasheet\nAll inputs use 100 nF except VREG in/out"
     (at 46.99 24.13 0)
+    (effects (font (size 1.27 1.27)) (justify left bottom))
+  )
+  (text "exact ordering may change for easier layout" (at 40.64 191.77 0)
     (effects (font (size 1.27 1.27)) (justify left bottom))
   )
@@
     )
   )
+  (global_label "MSFT_5V" (shape input) (at 171.45 139.7 90) (fields_autoplaced)
+    (effects (font (size 1.27 1.27)) (justify left))
+    (property "Intersheet References" "${INTERSHEET_REFS}" (id 0) (at 171.3706 129.304 90)
+      (effects (font (size 1.27 1.27)) (justify left) hide)
+    )
+  )
   (global_label "I2C0_SDA" (shape input) (at 181.61 71.12 0) (fields_autoplaced)
     (effects (font (size 1.27 1.27)) (justify left))
@@
     )
   )
+  (global_label "I2C0_SCL" (shape input) (at 29.21 181.61 180) (fields_autoplaced)
+    (effects (font (size 1.27 1.27)) (justify right))
+    (property "Intersheet References" "${INTERSHEET_REFS}" (id 0) (at 18.0279 181.6894 0)
+      (effects (font (size 1.27 1.27)) (justify right) hide)
+    )
+  )
   (global_label "MC_SCK" (shape input) (at 26.67 147.32 180) (fields_autoplaced)
     (effects (font (size 1.27 1.27)) (justify right))
@@
     )
   )
+  (global_label "TX" (shape input) (at 22.86 187.96 180) (fields_autoplaced)
+    (effects (font (size 1.27 1.27)) (justify right))
+    (property "Intersheet References" "${INTERSHEET_REFS}" (id 0) (at 18.2698 188.0394 0)
+      (effects (font (size 1.27 1.27)) (justify right) hide)
+    )
+  )
+  (global_label "I2C0_SDA" (shape input) (at 29.21 184.15 180) (fields_autoplaced)
+    (effects (font (size 1.27 1.27)) (justify right))
+    (property "Intersheet References" "${INTERSHEET_REFS}" (id 0) (at 17.9674 184.2294 0)
+      (effects (font (size 1.27 1.27)) (justify right) hide)
+    )
+  )
   (global_label "MC_SDA" (shape input) (at 26.67 144.78 180) (fields_autoplaced)
     (effects (font (size 1.27 1.27)) (justify right))
@@
     )
   )
+  (global_label "MSFT_VSYS" (shape input) (at 181.61 142.24 90) (fields_autoplaced)
+    (effects (font (size 1.27 1.27)) (justify left))
+    (property "Intersheet References" "${INTERSHEET_REFS}" (id 0) (at 181.5306 129.5459 90)
+      (effects (font (size 1.27 1.27)) (justify left) hide)
+    )
+  )
   (global_label "MC_SDA" (shape input) (at 172.72 43.18 0) (fields_autoplaced)
     (effects (font (size 1.27 1.27)) (justify left))
     (property "Intersheet References" "${INTERSHEET_REFS}" (id 0) (at 182.3902 43.1006 0)
       (effects (font (size 1.27 1.27)) (justify left) hide)
+    )
+  )
+  (global_label "RX" (shape input) (at 22.86 191.77 180) (fields_autoplaced)
+    (effects (font (size 1.27 1.27)) (justify right))
+    (property "Intersheet References" "${INTERSHEET_REFS}" (id 0) (at 17.9674 191.8494 0)
+      (effects (font (size 1.27 1.27)) (justify right) hide)
     )
   )
@@
     (pin "2")
   )
+  (symbol (lib_id "Connector:TestPoint") (at 74.93 170.18 90) (unit 1)
+    (in_bom yes) (on_board yes)
+    (property "Reference" "TP?" (id 0) (at 68.58 175.26 0)
+      (effects (font (size 1.27 1.27)) (justify left))
+    )
+    (property "Value" "TestPoint" (id 1) (at 71.12 180.34 0)
+      (effects (font (size 1.27 1.27)) (justify left))
+    )
+    (property "Footprint" "" (id 2) (at 74.93 165.1 0)
+      (effects (font (size 1.27 1.27)) hide)
+    )
+    (property "Datasheet" "~" (id 3) (at 74.93 165.1 0)
+      (effects (font (size 1.27 1.27)) hide)
+    )
+    (pin "1")
+  )
   (symbol (lib_id "Device:C_Small") (at 43.18 90.17 180) (unit 1)
     (in_bom yes) (on_board yes)
@@
     (pin "2")
   )
+  (symbol (lib_id "Connector:TestPoint") (at 69.85 167.64 90) (unit 1)
+    (in_bom yes) (on_board yes)
+    (property "Reference" "TP?" (id 0) (at 63.5 172.72 0)
+      (effects (font (size 1.27 1.27)) (justify left))
+    )
+    (property "Value" "TestPoint" (id 1) (at 66.04 177.8 0)
+      (effects (font (size 1.27 1.27)) (justify left))
+    )
+    (property "Footprint" "" (id 2) (at 69.85 162.56 0)
+      (effects (font (size 1.27 1.27)) hide)
+    )
+    (property "Datasheet" "~" (id 3) (at 69.85 162.56 0)
+      (effects (font (size 1.27 1.27)) hide)
+    )
+    (pin "1")
+  )
   (symbol (lib_id "Device:R_Small") (at 17.78 100.33 0) (unit 1)
     (in_bom yes) (on_board yes)
@@
       (effects (font (size 1.27 1.27)) (justify left))
     )
-    (property "Value" "470R" (id 1) (at 260.35 134.62 0)
+    (property "Value" "1K" (id 1) (at 260.35 134.62 0)
       (effects (font (size 1.27 1.27)) (justify left))
     )
@@
     )
     (property "Datasheet" "" (id 3) (at 273.05 140.97 0)
+      (effects (font (size 1.27 1.27)) hide)
+    )
+    (pin "1")
+  )
+  (symbol (lib_id "Connector:TestPoint") (at 132.08 177.8 0) (unit 1)
+    (in_bom yes) (on_board yes)
+    (property "Reference" "TP?" (id 0) (at 127 171.45 0)
+      (effects (font (size 1.27 1.27)) (justify left))
+    )
+    (property "Value" "TestPoint" (id 1) (at 121.92 173.99 0)
+      (effects (font (size 1.27 1.27)) (justify left))
+    )
+    (property "Footprint" "" (id 2) (at 137.16 177.8 0)
+      (effects (font (size 1.27 1.27)) hide)
+    )
+    (property "Datasheet" "~" (id 3) (at 137.16 177.8 0)
       (effects (font (size 1.27 1.27)) hide)
     )
@@
       (effects (font (size 1.27 1.27)) (justify left))
     )
-    (property "Value" "10K" (id 1) (at 128.27 180.34 90)
-      (effects (font (size 1.27 1.27)) (justify left))
-    )
+    (property "Value" "10K" (id 1) (at 124.46 181.61 90)
+      (effects (font (size 1.27 1.27)) (justify left))
+    )

Commit message: production version (2023)
Parts:
- removed D?: LED, symbol Device:LED
- removed J?: Micro_SD_Card, symbol Connector:Micro_SD_Card
- removed JP? (x2): HEADER-1X12, Adafruit Feather RP2040:1X12_ROUND, symbol Adafruit Feather RP2040-eagle-import:HEADER-1X12
- removed R? (x2): 10K, symbol Device:R_Small
- removed R? (x2): 4k7, symbol Device:R_Small
- removed R?: 1K, symbol Device:R_Small
- removed SW?: SWITCH_BOOTSEL, Adafruit Feather RP2040:EVQ-Q2, symbol Adafruit Feather RP2040-eagle-import:SWITCH_TACT_SMT
- removed SW?: SWITCH_RESET, Adafruit Feather RP2040:EVQ-Q2, symbol Adafruit Feather RP2040-eagle-import:SWITCH_TACT_SMT
- removed TP? (x2): TestPoint, symbol Connector:TestPoint
- removed Y?: 12MHz, symbol Device:Crystal_Small
- added C22: 100 nF 25V X7R, Capacitor_SMD:C_0402_1005Metric, symbol Device:C_Small
- added C23: 10 uF 16V X7R, Capacitor_SMD:C_0603_1608Metric_Pad1.08x0.95mm_HandSolder, symbol Device:C_Small
- added CONN1: SM04B-SRSS-TB(LF)(SN), RP2040:JST_SH4, symbol RP2040:STEMMA_I2C_QT
- added CONN2: SM04B-SRSS-TB(LF)(SN), RP2040:JST_SH4, symbol Adafruit Feather RP2040-eagle-import:STEMMA_I2C_QT
- added D2, D3, D4: Zener 3V3, Diode_SMD:D_MiniMELF, symbol Device:D_Zener_Small
- added J10, J7, J8, J9: header, Connector_PinHeader_2.54mm:PinHeader_1x01_P2.54mm_Vertical, symbol Connector:Conn_01x01_Female
- added J11: JST XH, Connector_JST:JST_XH_B4B-XH-A_1x04_P2.50mm_Vertical, symbol Connector:Conn_01x04_Female
- added J12: Micro_SD_Card, Connector_Card:microSD_HC_Molex_47219-2001, symbol Connector:Micro_SD_Card
- added J3, J4, J5: Conn_01x02_Female, Connector_PinHeader_2.54mm:PinHeader_1x02_P2.54mm_Vertical, symbol Connector:Conn_01x02_Female
- added J6: Conn_01x11_Female, Connector_Molex:Molex_KK-254_AE-6410-11A_1x11_P2.54mm_Vertical, symbol Connector:Conn_01x11_Female
- added Q1: BSS138, Package_TO_SOT_SMD:SOT-23, symbol Transistor_FET:AO3400A
- added R10, R11, R17, R20, R25, R28, R29, R7, R8, R9: 330, Resistor_SMD:R_0603_1608Metric, symbol Device:R_Small
- added R13: 200K, Capacitor_SMD:C_0402_1005Metric_Pad0.74x0.62mm_HandSolder, symbol Device:R_Small
- added R14, R15, R22, R30, R36, R37: 27R, Capacitor_SMD:C_0402_1005Metric_Pad0.74x0.62mm_HandSolder, symbol Device:R_Small
- added R16, R34: 10K, Capacitor_SMD:C_0402_1005Metric_Pad0.74x0.62mm_HandSolder, symbol Device:R_Small
- added R21, R26, R33, R35: 4K7, Resistor_SMD:R_0603_1608Metric_Pad0.98x0.95mm_HandSolder, symbol Device:R_Small
- added R23, R31, R32: 110K, Capacitor_SMD:C_0603_1608Metric, symbol Device:R_Small
- added R24, R27, R39: 1M, Capacitor_SMD:C_0402_1005Metric_Pad0.74x0.62mm_HandSolder, symbol Device:R_Small
- added SW1, SW2, SW3: SW_SPST, Button_Switch_SMD:SW_Push_1P1T_NO_6x6mm_H9.5mm, symbol Switch:SW_SPST
- added U7: TPD4EUSB30, Package_SON:USON-10_2.5x1.0mm_P0.5mm, symbol Power_Protection:TPD4EUSB30
- added Y2: 12MHz X322512MSB4SI, Crystal:Crystal_SMD_3225-4Pin_3.2x2.5mm, symbol Device:Crystal_GND24_Small
- C10, C11, C12, C13, C14, C15, C16, C20, C21, C24: renamed from C?; value 100 nF -> 100 nF 25V X7R; footprint (none) -> Capacitor_SMD:C_0402_1005Metric; JCLPCB (none) -> C307331; Vendor (none) -> C307331
- C17, C18, C19: renamed from C?; value 1 uF -> 1 uF 50V X5R; footprint (none) -> Capacitor_SMD:C_0603_1608Metric; JCLPCB (none) -> C15849; Vendor (none) -> C15849
- C25, C26: renamed from C?; value 22pF -> 33 pF 6V C0G; footprint (none) -> Capacitor_SMD:C_0402_1005Metric_Pad0.74x0.62mm_HandSolder; JCLPCB (none) -> C1562; Vendor (none) -> C1562
- IC1: renamed from IC?; footprint Adafruit Feather RP2040:QFN56_7MM_REDUCEDEPAD -> RP2040:QFN56_7MM_REDUCEDEPAD; JCLPCB (none) -> C2040; Vendor (none) -> C2040
- R12: renamed from R?; value 10K -> 1K; footprint (none) -> Capacitor_SMD:C_0402_1005Metric_Pad0.74x0.62mm_HandSolder; JCLPCB (none) -> C11702; Vendor (none) -> C11702
- R18, R19: renamed from R?; footprint (none) -> Capacitor_SMD:C_0402_1005Metric_Pad0.74x0.62mm_HandSolder; JCLPCB (none) -> C25100; Vendor (none) -> C25100
- R38: renamed from R?; footprint (none) -> Capacitor_SMD:C_0402_1005Metric_Pad0.74x0.62mm_HandSolder; JCLPCB (none) -> C11702; Vendor (none) -> C11702
- R5, R6: renamed from R?; footprint (none) -> Capacitor_SMD:C_0402_1005Metric_Pad0.74x0.62mm_HandSolder; JCLPCB (none) -> C25744; Vendor (none) -> C25744
- TP2: renamed from TP?; footprint (none) -> TestPoint:TestPoint_Pad_D1.5mm
- U6: renamed from U?; value W25Q128JVS -> W25Q16JVS; JCLPCB (none) -> C82317; Vendor (none) -> C82317
Connections:
- net +3V3: now also U6.8 (VCC), C23.2, CONN1.2 (V+), CONN2.2 (V+), J12.4 (VDD), J6.3 (Pin_3), Q1.1 (G), R16.2, R21.1, R23.1, R26.1, R33.1, R34.1, R35.1
- net +5V: now also C22.1, J11.2 (Pin_2), R31.1
- net GND: now also C16.1, C17.1, C22.2, C23.1, CONN1.1 (GND), CONN1.MT1 (MT), CONN1.MT2 (MT), CONN2.1 (GND), CONN2.MT1 (MT), CONN2.MT2 (MT), D2.2 (A), D3.2 (A), D4.2 (A), J11.1 (Pin_1), J11.4 (Pin_4), J12.6 (VSS), J12.9 (SHIELD), J6.6 (Pin_6), J6.9 (Pin_9), R13.2, R24.1, R27.1, R32.2, SW1.2 (B), SW3.2 (B), U7.3 (GND), U7.8 (GND), Y2.2, Y2.4
- net GPIO18: now also J12.5 (CLK)
- net GPIO19: now also J12.3 (CMD)
- net GPIO20: now also J12.7 (DAT0), R34.2
- net GPIO21: now also J12.8 (DAT1), J7.1 (Pin_1)
- net GPIO22: now also J12.1 (DAT2), J8.1 (Pin_1)
- net GPIO26: now also J6.8 (Pin_8)
- net GPIO27: now also J6.7 (Pin_7)
- net GPIO28: now also D2.1 (K), R9.1
- net I2C0_SCL: now also CONN1.4 (SCL), J4.2 (Pin_2), R37.1; no longer IC1.16 (GPIO13)
- net I2C0_SDA: now also CONN1.3 (SDA), J4.1 (Pin_1), R36.2; no longer IC1.15 (GPIO12)
- net MC_SCK: now also CONN2.4 (SCL), J3.1 (Pin_1), R30.1; no longer IC1.5 (GPIO3)
- net MC_SDA: now also CONN2.3 (SDA), J3.2 (Pin_2), R22.2; no longer IC1.4 (GPIO2)
- net MSFT_5V: now also R25.2, R27.2
- net RESET: now also SW1.1 (A)
- net RX: now also J6.2 (Pin_2), R15.1; no longer IC1.3 (GPIO1)
- net SWCLK: now also J5.1 (Pin_1)
- net SWDIO: now also J5.2 (Pin_2)
- net TX: now also J6.1 (Pin_1), R14.2; no longer IC1.2 (GPIO0)
- net XIN: now also Y2.3
- net at C25.1, R38.1: now also Y2.1
- net QSPI_SD1: now reaches IC1.55 (QSPI_SD1), U6.2 (DO(IO1))
- net QSPI_SD2: now reaches IC1.54 (QSPI_SD2), U6.3 (IO2)
- net QSPI_SD0: now reaches IC1.53 (QSPI_SD0), U6.5 (DI(IO0))
- net QSPI_SD3: now reaches IC1.51 (QSPI_SD3), U6.7 (IO3)
- net BTSEL: now reaches R12.1, TP2.1
- net BTSEL: now also SW3.1 (A)
- net G11: now reaches IC1.14 (GPIO11)
- net G11: now also R17.2, U7.5 (D2-)
- net 5V_HEAD1: now reaches IC1.17 (GPIO14)
- net 5V_HEAD1: now also R13.1, SW2.1 (A)
- net 5V_HEAD0: now reaches IC1.18 (GPIO15)
- net 5V_HEAD0: now also R20.1
- net INOKB GPIO16: now reaches IC1.27 (GPIO16)
- net INOKB GPIO16: now also R39.2
- net GPIO23: now reaches IC1.35 (GPIO23)
- net GPIO23: now also J12.2 (DAT3/CD)
- net at IC1.36 (GPIO24): now also R8.1
- net GPIO29: now reaches IC1.41 (GPIO29/AD3)
- net GPIO29: now also D3.1 (K), R10.1
- net GPIO10 renamed GP10
- net GP10: now also J10.1 (Pin_1), R25.1, U7.4 (D2+)
- net GPIO17: no longer names the net of IC1.28 (GPIO17)
- net GPIO17: now also J9.1 (Pin_1), R28.1
- net GPIO4 renamed GP4_MS
- net GP4_MS: now also R24.2, R29.1
- net GPIO5 renamed SYS_HEAD3
- net GPIO6 renamed SYS_HEAD2
- net GPIO7 renamed GP7
- net GP7: now also D4.1 (K), R11.1
- net GPIO8 renamed GP8
- net GP8: now also R33.2, R36.1, U7.1 (D1+)
- net GPIO9 renamed GP9
- net GP9: now also R35.2, R37.2, U7.2 (D1-)
- net LED GP25: no longer names the net of IC1.37 (GPIO25)
- net LED GP25: now also R7.2
- new net: IC1.2 (GPIO0), R14.1
- new net: IC1.4 (GPIO2), R21.2, R22.1
- new net: R16.1, SW2.2 (B)
- new net: J6.4 (Pin_4), R10.2
- new net: J6.5 (Pin_5), R9.2
- new net: IC1.5 (GPIO3), R26.2, R30.2
- new net: IC1.3 (GPIO1), R15.2
- new net 5V Logic: J11.3 (Pin_3), Q1.3 (D), R31.2
- new net 5V_HEAD2: IC1.16 (GPIO13)
- new net 5V_HEAD3: IC1.15 (GPIO12)
- new net 5V_HEAD4: R17.1
- new net GPIO24: J6.11 (Pin_11), R8.2
- new net GPIO25: J6.10 (Pin_10), R7.1
- new net INOKB: R39.1
- new net LVS: Q1.2 (S), R20.2, R23.2
- new net MSFT_BATT: R28.2, R32.1
- new net MSFT_VSV: R29.2
- new net SYS_HEAD1: R11.2
- no-connect marks 9 -> 0
Other:
- note added: "5V Logic Level Shifter"
- note added: "Adding protection to just a few of the signal pins"
- note added: "Crystal caps are 'effectively in series' (load capacitance - stray cap ~ 4pF) * 2 = cap to use but most places say 'anything 18 - 33 pF will probably work'"
- note added: "The constraints our SD PIO software puts upon us is that the four data signals must be connected to contiguous GPIOs. The CLK and CMD signals can go anywhere (excepting also SPI requirements) pullup here on MISO, some debate if others are required"
- note added: "Useful: https://blog.thea.codes/starfish-a-control-board-with-the-rp2040/"
- note removed: "Also seen 27pF, 15pF"
- note removed: "Not sure about this 1uF on Flash"
- note removed: "exact ordering may change for easier layout"
- moved on the sheet: C20, C24, C25, C26, R12, R38, TP2
